Commit message: Update Hunter SE robot description

File: ugv_gazebo_sim/hunter_se/hunter_se_description/urdf/hunter_se.xacro (robot description, xacro)
@@ -3,4 +3,11 @@
     xmlns:xacro="http://ros.org/wiki/xacro">
     <xacro:include filename="$(find hunter_se_description)/urdf/lidar_3d.xacro"/>
+    <!-- ===================== Footprint (ground-projected root) ===================== -->
+    <link name="base_footprint"/>
+    <joint name="base_footprint_joint" type="fixed">
+        <parent link="base_footprint"/>
+        <child link="base_link"/>
+        <origin xyz="0 0 0.2955" rpy="0 0 0"/>
+    </joint>
     <!-- ===================== Base ===================== -->
     <link name="base_link">
@@ -185,20 +192,58 @@
         <dynamics damping="0.0" friction="0.1"/>
     </joint>
+    <!-- ===================== Colors (gz-sim) ===================== -->
+    <gazebo reference="base_link">
+        <visual>
+            <material>
+                <ambient>0.752941 0.752941 0.752941 1</ambient>
+                <diffuse>0.752941 0.752941 0.752941 1</diffuse>
+                <specular>0.2 0.2 0.2 1</specular>
+            </material>
+        </visual>
+    </gazebo>
     <!-- ===================== Wheel surface friction ===================== -->
     <gazebo reference="fr_left_link">
         <mu1>0.8</mu1><mu2>0.8</mu2><kp>500000.0</kp><kd>10.0</kd>
         <minDepth>0.001</minDepth><maxVel>0.1</maxVel><fdir1>1 0 0</fdir1>
+        <visual>
+            <material>
+                <ambient>0.223529 0.223529 0.223529 1</ambient>
+                <diffuse>0.223529 0.223529 0.223529 1</diffuse>
+                <specular>0.1 0.1 0.1 1</specular>
+            </material>
+        </visual>
     </gazebo>
     <gazebo reference="fr_right_link">
         <mu1>0.8</mu1><mu2>0.8</mu2><kp>500000.0</kp><kd>10.0</kd>
         <minDepth>0.001</minDepth><maxVel>0.1</maxVel><fdir1>1 0 0</fdir1>
+        <visual>
+            <material>
+                <ambient>0.223529 0.223529 0.223529 1</ambient>
+                <diffuse>0.223529 0.223529 0.223529 1</diffuse>
+                <specular>0.1 0.1 0.1 1</specular>
+            </material>
+        </visual>
     </gazebo>
     <gazebo reference="re_left_link">
         <mu1>0.8</mu1><mu2>10</mu2><kp>500000.0</kp><kd>10.0</kd>
         <minDepth>0.001</minDepth><maxVel>0.1</maxVel><fdir1>1 0 0</fdir1>
+        <visual>
+            <material>
+                <ambient>0.223529 0.223529 0.223529 1</ambient>
+                <diffuse>0.223529 0.223529 0.223529 1</diffuse>
+                <specular>0.1 0.1 0.1 1</specular>
+            </material>
+        </visual>
     </gazebo>
     <gazebo reference="re_right_link">
         <mu1>0.8</mu1><mu2>10</mu2><kp>500000.0</kp><kd>10.0</kd>
         <minDepth>0.001</minDepth><maxVel>0.1</maxVel><fdir1>1 0 0</fdir1>
+        <visual>
+            <material>
+                <ambient>0.223529 0.223529 0.223529 1</ambient>
+                <diffuse>0.223529 0.223529 0.223529 1</diffuse>
+                <specular>0.1 0.1 0.1 1</specular>
+            </material>
+        </visual>
     </gazebo>
     <!-- ===================== Gazebo (gz-sim) plugins ===================== -->
@@ -231,5 +276,5 @@
         <plugin filename="gz-sim-odometry-publisher-system" name="gz::sim::systems::OdometryPublisher">
             <odom_frame>odom</odom_frame>
-            <robot_base_frame>base_link</robot_base_frame>
+            <robot_base_frame>base_footprint</robot_base_frame>
             <odom_publish_frequency>50</odom_publish_frequency>
             <odom_topic>odom</odom_topic>

File: ugv_gazebo_sim/hunter_se/hunter_se_description/urdf/lidar_3d.xacro (robot description, xacro)
@@ -2,4 +2,32 @@
 <robot xmlns:xacro="http://ros.org/wiki/xacro">
     <xacro:macro name="lidar_3d" params="parent:=base_link">
+        <!-- Support mast mounting the lidar to the chassis -->
+        <link name="lidar_mast_link">
+            <inertial>
+                <mass value="0.2"/>
+                <origin xyz="0 0 0.1075" rpy="0 0 0"/>
+                <inertia ixx="1e-3" ixy="0" ixz="0" iyy="1e-3" iyz="0" izz="1e-4"/>
+            </inertial>
+            <visual>
+                <origin xyz="0 0 0.1075" rpy="0 0 0"/>
+                <geometry>
+                    <cylinder radius="0.025" length="0.215"/>
+                </geometry>
+                <material name="mast_material">
+                    <color rgba="0 0 0 1"/>
+                </material>
+            </visual>
+            <collision>
+                <origin xyz="0 0 0.1075" rpy="0 0 0"/>
+                <geometry>
+                    <cylinder radius="0.025" length="0.215"/>
+                </geometry>
+            </collision>
+        </link>
+        <joint name="lidar_mast_joint" type="fixed">
+            <parent link="${parent}"/>
+            <child link="lidar_mast_link"/>
+            <origin xyz="0 0 0" rpy="0 0 0"/>
+        </joint>
         <link name="velodyne_link">
             <inertial>
@@ -25,9 +53,25 @@
         </link>
         <joint name="velodyne_joint" type="fixed">
-            <parent link="${parent}"/>
+            <parent link="lidar_mast_link"/>
             <child link="velodyne_link"/>
             <origin xyz="0 0 0.25" rpy="0 0 0"/>
         </joint>
+        <gazebo reference="lidar_mast_link">
+            <visual>
+                <material>
+                    <ambient>0 0 0 1</ambient>
+                    <diffuse>0 0 0 1</diffuse>
+                    <specular>0.05 0.05 0.05 1</specular>
+                </material>
+            </visual>
+        </gazebo>
         <gazebo reference="velodyne_link">
+            <visual>
+                <material>
+                    <ambient>0.3 0.3 0.3 1</ambient>
+                    <diffuse>0.3 0.3 0.3 1</diffuse>
+                    <specular>0.1 0.1 0.1 1</specular>
+                </material>
+            </visual>
             <sensor name="velodyne" type="gpu_lidar">
                 <gz_frame_id>velodyne_link</gz_frame_id>
